Commit message: Add an optional wrist-mounted RGB-D camera
New camera_mount argument (stand | wrist, default stand) selects where the
simulated D435 is mounted. The D435 xacro is now a macro, the stand moved to
its own file, and the wrist camera sits on gripper_base looking along the
fingers with a 0.1 m near clip. Its topics are bridged under /camera_wrist.
The camera inertia is now computed from its size.

File: src/pnp_cobot_ros2/pnp_cobot_description/urdf/robots/pnp_cobot_280.urdf.xacro (robot description, xacro)
@@ -9,4 +9,5 @@
     <xacro:arg name="prefix" default=""/>
     <xacro:arg name="use_camera" default="false"/>
+    <xacro:arg name="camera_mount" default="stand"/>
     <xacro:arg name="use_gazebo" default="false"/>
     <xacro:arg name="use_gripper" default="true"/>
@@ -53,4 +54,27 @@
       flange_link="$(arg flange_link)"
       use_gazebo="$(arg use_gazebo)"/>
-    <xacro:include filename="$(find pnp_cobot_description)/urdf/sensors/intel_rgbd_cam_d435.urdf.xacro"/>
+    <!-- RGB-D camera: fixed on a stand next to the robot, or on the wrist (eye-in-hand) -->
+    <xacro:if value="$(arg use_camera)">
+        <xacro:include filename="$(find pnp_cobot_description)/urdf/sensors/intel_rgbd_cam_d435.urdf.xacro"/>
+        <xacro:property name="current_camera_mount" value="$(arg camera_mount)"/>
+        <xacro:if value="${current_camera_mount == 'stand'}">
+            <xacro:include filename="$(find pnp_cobot_description)/urdf/mech/camera_stand.urdf.xacro"/>
+            <xacro:camera_stand parent="$(arg prefix)$(arg base_link)">
+                <origin xyz="0.22 -0.30 0" rpy="0 0 0"/>
+            </xacro:camera_stand>
+            <xacro:intel_rgbd_cam_d435 name="camera_head" parent="torso_link"
+                                       use_gazebo="$(arg use_gazebo)">
+                <origin xyz="0 0.01 0.50" rpy="0 ${radians(25)} ${pi/2}"/>
+            </xacro:intel_rgbd_cam_d435>
+        </xacro:if>
+        <!-- gripper_base frame: +y towards the fingertips, x across the fingers. The camera sits
+             on the +z side of the gripper and looks along +y. Its depth range starts at 0.1 m
+             like a D435 at this resolution, so the fingertips (~6 cm ahead) are not in the cloud. -->
+        <xacro:if value="${current_camera_mount == 'wrist'}">
+            <xacro:intel_rgbd_cam_d435 name="camera_wrist" parent="$(arg prefix)gripper_base"
+                                       use_gazebo="$(arg use_gazebo)" near_clip="0.1">
+                <origin xyz="0 0 0.03" rpy="0 0 ${pi/2}"/>
+            </xacro:intel_rgbd_cam_d435>
+        </xacro:if>
+    </xacro:if>
 </robot>

File: src/pnp_cobot_ros2/pnp_cobot_description/urdf/sensors/intel_rgbd_cam_d435.urdf.xacro (robot description, xacro)
@@ -1,66 +1,27 @@
 <?xml version="1.0"?>
+<!--
+  Intel RealSense D435 RGB-D camera: body link, depth/infra/color frames and the Gazebo sensor.
+  Modified by: Souvik Roy <sroyy57@gmail.com> (2026) — turned into a macro so the camera can be
+  mounted on the stand or on the wrist; box inertia computed from the camera size.
+  Links are named after `name`: <name>_link (x forward, z up), <name>_depth_optical_frame, ...
+  The Gazebo topic is `name` (<name>/points, <name>/image, <name>/depth_image, <name>/camera_info).
+-->
 <robot xmlns:xacro="http://www.ros.org/wiki/xacro">
-  <xacro:arg name="use_camera" default="true"/>
-  <xacro:arg name="use_gazebo" default="true"/>
-  <xacro:arg name="prefix" default=""/>
-  <xacro:if value="${'true' == '$(arg use_camera)' and 'true' == '$(arg use_gazebo)'}">
-    <xacro:property name="M_PI" value="3.1415926535897931" />
+  <xacro:macro name="intel_rgbd_cam_d435" params="name parent use_gazebo near_clip:=0.05 *origin">
     <xacro:property name="d435_cam_width" value="0.090"/>
     <xacro:property name="d435_cam_height" value="0.025"/>
     <xacro:property name="d435_cam_depth" value="0.02505"/>
+    <xacro:property name="d435_cam_mass" value="0.072"/>
     <xacro:property name="d435_cam_depth_to_infra1_offset" value="0.0"/>
     <xacro:property name="d435_cam_depth_to_infra2_offset" value="-0.050"/>
     <xacro:property name="d435_cam_depth_to_color_offset" value="0.015"/>
-    <xacro:property name="camera_tilt_angle_deg" value="25"/>
-    <link name="torso_link">
-      <inertial>
-        <origin xyz="0 0 0.50" />
-        <mass value="2.5" />
-        <inertia ixx="0.8" ixy="0.0" ixz="0.0" iyy="0.8" iyz="0.0" izz="0.8" />
-      </inertial>
-      <visual name="holder">
-        <origin xyz="0 0 0.25" rpy="0 0 0" />
-        <material name="LightGrey">
-          <color rgba="0.7 0.7 0.7 1.0"/>
-        </material>
-        <geometry>
-          <cylinder radius="0.005" length="0.5"/>
-        </geometry>
-      </visual>
-      <visual name="base">
-        <origin xyz="0 0 0" rpy="0 0 0" />
-        <material name="LightGrey">
-          <color rgba="0.7 0.7 0.7 1.0"/>
-        </material>
-        <geometry>
-          <box size="0.15 0.10 0.06" />
-        </geometry>
-      </visual>
-      <collision name="holder">
-        <origin xyz="0 0 0.25" rpy="0 0 0" />
-        <geometry>
-          <cylinder radius="0.005" length="0.6"/>
-        </geometry>
-      </collision>
-      <collision name="base">
-        <origin xyz="0 0 0.0" rpy="0 0 0" />
-        <geometry>
-          <box size="0.15 0.10 0.06" />
-        </geometry>
-      </collision>
-    </link>
-    <joint name="$(arg prefix)base_link_to_torso_link" type="fixed">
-      <parent link="$(arg prefix)base_link"/>
-      <child link="torso_link"/>
-      <origin xyz="0.22 -0.30 0" rpy="0 0 0"/>
+    <joint name="${name}_joint" type="fixed">
+      <parent link="${parent}"/>
+      <child link="${name}_link"/>
+      <xacro:insert_block name="origin"/>
     </joint>
-    <joint name="camera_head_joint" type="fixed">
-      <parent link="torso_link"/>
-      <child link="camera_head_link" />
-      <origin xyz="0 0.01 0.50" rpy="0.0 ${camera_tilt_angle_deg * M_PI / 180} ${M_PI/2}"/>
-    </joint>
-    <link name="camera_head_link">
+    <link name="${name}_link">
       <visual>
-        <origin xyz="0 0 0" rpy="${M_PI/2} 0.0 ${M_PI/2}"/>
+        <origin xyz="0 0 0" rpy="${pi/2} 0.0 ${pi/2}"/>
         <geometry>
           <mesh filename="file://$(find pnp_cobot_description)/meshes/d435/visual/d435.stl" />
@@ -77,77 +38,82 @@
       </collision>
       <inertial>
-        <mass value="0.072" />
+        <mass value="${d435_cam_mass}" />
         <origin xyz="0 0 0" />
-        <inertia ixx="0.003881243" ixy="0.0" ixz="0.0" iyy="0.000498940" iyz="0.0" izz="0.003879257" />
+        <inertia
+          ixx="${d435_cam_mass / 12 * (d435_cam_width**2 + d435_cam_height**2)}" ixy="0.0" ixz="0.0"
+          iyy="${d435_cam_mass / 12 * (d435_cam_depth**2 + d435_cam_height**2)}" iyz="0.0"
+          izz="${d435_cam_mass / 12 * (d435_cam_depth**2 + d435_cam_width**2)}" />
       </inertial>
     </link>
-    <joint name="camera_head_depth_joint" type="fixed">
+    <joint name="${name}_depth_joint" type="fixed">
       <origin xyz="0 0 0" rpy="0 0 0"/>
-      <parent link="camera_head_link"/>
-      <child link="camera_head_depth_frame" />
+      <parent link="${name}_link"/>
+      <child link="${name}_depth_frame" />
     </joint>
-    <link name="camera_head_depth_frame"/>
-    <joint name="camera_head_depth_optical_joint" type="fixed">
-      <origin xyz="0 0 0" rpy="${-M_PI/2} 0 ${-M_PI/2}" />
-      <parent link="camera_head_depth_frame" />
-      <child link="camera_head_depth_optical_frame" />
+    <link name="${name}_depth_frame"/>
+    <joint name="${name}_depth_optical_joint" type="fixed">
+      <origin xyz="0 0 0" rpy="${-pi/2} 0 ${-pi/2}" />
+      <parent link="${name}_depth_frame" />
+      <child link="${name}_depth_optical_frame" />
     </joint>
-    <link name="camera_head_depth_optical_frame"/>
-    <joint name="camera_head_infra1_joint" type="fixed">
+    <link name="${name}_depth_optical_frame"/>
+    <joint name="${name}_infra1_joint" type="fixed">
       <origin xyz="0 ${d435_cam_depth_to_infra1_offset} 0" rpy="0 0 0" />
-      <parent link="camera_head_link" />
-      <child link="camera_head_infra1_frame" />
+      <parent link="${name}_link" />
+      <child link="${name}_infra1_frame" />
     </joint>
-    <link name="camera_head_infra1_frame"/>
-    <joint name="camera_head_infra1_optical_joint" type="fixed">
-      <origin xyz="0 0 0" rpy="${-M_PI/2} 0 ${-M_PI/2}" />
-      <parent link="camera_head_infra1_frame" />
-      <child link="camera_head_infra1_optical_frame" />
+    <link name="${name}_infra1_frame"/>
+    <joint name="${name}_infra1_optical_joint" type="fixed">
+      <origin xyz="0 0 0" rpy="${-pi/2} 0 ${-pi/2}" />
+      <parent link="${name}_infra1_frame" />
+      <child link="${name}_infra1_optical_frame" />
     </joint>
-    <link name="camera_head_infra1_optical_frame"/>
-    <joint name="camera_head_infra2_joint" type="fixed">
+    <link name="${name}_infra1_optical_frame"/>
+    <joint name="${name}_infra2_joint" type="fixed">
       <origin xyz="0 ${d435_cam_depth_to_infra2_offset} 0" rpy="0 0 0" />
-      <parent link="camera_head_link" />
-      <child link="camera_head_infra2_frame" />
+      <parent link="${name}_link" />
+      <child link="${name}_infra2_frame" />
     </joint>
-    <link name="camera_head_infra2_frame"/>
-    <joint name="camera_head_infra2_optical_joint" type="fixed">
-      <origin xyz="0 0 0" rpy="${-M_PI/2} 0 ${-M_PI/2}" />
-      <parent link="camera_head_infra2_frame" />
-      <child link="camera_head_infra2_optical_frame" />
+    <link name="${name}_infra2_frame"/>
+    <joint name="${name}_infra2_optical_joint" type="fixed">
+      <origin xyz="0 0 0" rpy="${-pi/2} 0 ${-pi/2}" />
+      <parent link="${name}_infra2_frame" />
+      <child link="${name}_infra2_optical_frame" />
     </joint>
-    <link name="camera_head_infra2_optical_frame"/>
-    <joint name="camera_head_color_joint" type="fixed">
+    <link name="${name}_infra2_optical_frame"/>
+    <joint name="${name}_color_joint" type="fixed">
       <origin xyz="0 ${d435_cam_depth_to_color_offset} 0" rpy="0 0 0" />
-      <parent link="camera_head_link" />
-      <child link="camera_head_color_frame" />
+      <parent link="${name}_link" />
+      <child link="${name}_color_frame" />
     </joint>
-    <link name="camera_head_color_frame"/>
-    <joint name="camera_head_color_optical_joint" type="fixed">
-      <origin xyz="0 0 0" rpy="${-M_PI/2} 0 ${-M_PI/2}" />
-      <parent link="camera_head_color_frame" />
-      <child link="camera_head_color_optical_frame" />
+    <link name="${name}_color_frame"/>
+    <joint name="${name}_color_optical_joint" type="fixed">
+      <origin xyz="0 0 0" rpy="${-pi/2} 0 ${-pi/2}" />
+      <parent link="${name}_color_frame" />
+      <child link="${name}_color_optical_frame" />
     </joint>
-    <link name="camera_head_color_optical_frame"/>
-    <gazebo reference="camera_head_link">
-      <sensor name="camera_head" type="rgbd_camera">
-        <camera>
-          <horizontal_fov>1.5184</horizontal_fov>
-          <image>
-            <width>424</width>
-            <height>240</height>
-          </image>
-          <clip>
-            <near>0.05</near>
-            <far>1.5</far>
-          </clip>
-        </camera>
-        <always_on>1</always_on>
-        <ignition_frame_id>camera_head_link</ignition_frame_id>
-        <topic>camera_head</topic>
-        <update_rate>5</update_rate>
-        <visualize>true</visualize>
-      </sensor>
-    </gazebo>
-  </xacro:if>
+    <link name="${name}_color_optical_frame"/>
+    <xacro:if value="${use_gazebo}">
+      <gazebo reference="${name}_link">
+        <sensor name="${name}" type="rgbd_camera">
+          <camera>
+            <horizontal_fov>1.5184</horizontal_fov>
+            <image>
+              <width>424</width>
+              <height>240</height>
+            </image>
+            <clip>
+              <near>${near_clip}</near>
+              <far>1.5</far>
+            </clip>
+          </camera>
+          <always_on>1</always_on>
+          <ignition_frame_id>${name}_link</ignition_frame_id>
+          <topic>${name}</topic>
+          <update_rate>5</update_rate>
+          <visualize>true</visualize>
+        </sensor>
+      </gazebo>
+    </xacro:if>
+  </xacro:macro>
 </robot>
